Commit message: feat: update (from pinocchino 2.6.3 to 3.31)

File: ur5/urdf/ur5_robot3.urdf (robot description, URDF)
Before this commit: robot ur5, 8 links, 7 joints
Links:
- added link base, mass 0
- added link tool0, mass 0
- added link world
- link base_link: geometry collision mesh filename=package://ur5/meshes/collision/base.stl; visual mesh filename=package://ur5/meshes/visual/base.dae
- link ee_link: mass 0.1 -> 0; geometry collision box size=0.01 0.01 0.01
- link forearm_link: geometry collision mesh filename=package://ur5/meshes/collision/forearm.stl; visual mesh filename=package://ur5/meshes/visual/forearm.dae
- link shoulder_link: geometry collision mesh filename=package://ur5/meshes/collision/shoulder.stl; visual mesh filename=package://ur5/meshes/visual/shoulder.dae
- link upper_arm_link: geometry collision mesh filename=package://ur5/meshes/collision/upperarm.stl; visual mesh filename=package://ur5/meshes/visual/upperarm.dae
- link wrist_1_link: geometry collision mesh filename=package://ur5/meshes/collision/wrist1.stl; visual mesh filename=package://ur5/meshes/visual/wrist1.dae
- link wrist_2_link: geometry collision mesh filename=package://ur5/meshes/collision/wrist2.stl; visual mesh filename=package://ur5/meshes/visual/wrist2.dae
- link wrist_3_link: geometry collision mesh filename=package://ur5/meshes/collision/wrist3.stl; visual mesh filename=package://ur5/meshes/visual/wrist3.dae
Joints:
- added joint base_link-base_fixed_joint: type fixed, parent base_link, child base, origin xyz=0 0 0 rpy=0 0 -3.14159265359
- added joint world_joint: type fixed, parent world, child base_link, origin xyz=0.0 0.0 0.0 rpy=0.0 0.0 0.0
- added joint wrist_3_link-tool0_fixed_joint: type fixed, parent wrist_3_link, child tool0, origin xyz=0 0.0823 0 rpy=-1.57079632679 0 0
- joint ee_fixed_joint: origin xyz=0.0 0.18 0.0 rpy=1.570796325 0.0 0.0 -> xyz=0.0 0.0823 0.0 rpy=0.0 0.0 1.57079632679
- joint elbow_joint: limit lower=-6.2831853 upper=6.2831853 effort=150.0 velocity=3.15 -> lower=-3.14159265359 upper=3.14159265359 effort=150.0 velocity=3.15
- joint shoulder_lift_joint: limit lower=-6.2831853 upper=6.2831853 effort=150.0 velocity=3.15 -> lower=-6.28318530718 upper=6.28318530718 effort=150.0 velocity=3.15; origin xyz=0.0 0.13585 0.0 rpy=0.0 1.570796325 0.0 -> xyz=0.0 0.13585 0.0 rpy=0.0 1.57079632679 0.0
- joint shoulder_pan_joint: limit lower=-6.2831853 upper=6.2831853 effort=150.0 velocity=3.15 -> lower=-6.28318530718 upper=6.28318530718 effort=150.0 velocity=3.15
- joint wrist_1_joint: limit lower=-6.2831853 upper=6.2831853 effort=28.0 velocity=3.2 -> lower=-6.28318530718 upper=6.28318530718 effort=28.0 velocity=3.2; origin xyz=0.0 0.0 0.39225 rpy=0.0 1.570796325 0.0 -> xyz=0.0 0.0 0.39225 rpy=0.0 1.57079632679 0.0
- joint wrist_2_joint: limit lower=-6.2831853 upper=6.2831853 effort=28.0 velocity=3.2 -> lower=-6.28318530718 upper=6.28318530718 effort=28.0 velocity=3.2
- joint wrist_3_joint: limit lower=-6.2831853 upper=6.2831853 effort=28.0 velocity=3.2 -> lower=-6.28318530718 upper=6.28318530718 effort=28.0 velocity=3.2
